File: src/buttons_tac.kicad_sch (KiCad schematic)
At the start: 41 parts, among them J3 Micro_SD_Card, Q2 Q_NMOS_GSD, Q5 NPN, SW5 SW_Push, SW6 SW_Push, SW7 SW_Push, SW8 SW_Push, U10 IRM-H6xxT

Commit message: footprints adicionados componentes elétricos GPIOS
Parts:
- R23, R24: footprint (none) -> Resistor_SMD:R_0402_1005Metric
Changed lines of the file:
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@@
 			)
 		)
-		(property "Footprint" ""
+		(property "Footprint" "Resistor_SMD:R_0402_1005Metric"
 			(at 118.11 43.18 0)
 			(effects
@@
 			)
 		)
-		(property "Footprint" ""
+		(property "Footprint" "Resistor_SMD:R_0402_1005Metric"
 			(at 207.01 62.23 0)
 			(effects
